File: Snail/Snail.kicad_pcb (KiCad board)
At the start: 0 parts

Commit message: Board configuration
Other:
- copper layers 0 -> 2
Changed lines of the file:
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@@
 (kicad_pcb
-  (version 20260206)
-  (generator "pcbnew")
-  (generator_version "10.0"))
+	(version 20260206)
+	(generator "pcbnew")
+	(generator_version "10.0")
+	(general
+		(thickness 1.6)
+		(legacy_teardrops no)
+	)
+	(paper "A4")
+	(layers
+		(0 "F.Cu" signal)
+		(2 "B.Cu" signal)
+		(9 "F.Adhes" user "F.Adhesive")
+		(11 "B.Adhes" user "B.Adhesive")
+		(13 "F.Paste" user)
+		(15 "B.Paste" user)
+		(5 "F.SilkS" user "F.Silkscreen")
+		(7 "B.SilkS" user "B.Silkscreen")
+		(1 "F.Mask" user)
+		(3 "B.Mask" user)
+		(17 "Dwgs.User" user "User.Drawings")
+		(19 "Cmts.User" user "User.Comments")
+		(21 "Eco1.User" user "User.Eco1")
+		(23 "Eco2.User" user "User.Eco2")
+		(25 "Edge.Cuts" user)
+		(27 "Margin" user)
+		(31 "F.CrtYd" user "F.Courtyard")
+		(29 "B.CrtYd" user "B.Courtyard")
+		(35 "F.Fab" user)
+		(33 "B.Fab" user)
+		(39 "User.1" user)
+		(41 "User.2" user)
+		(43 "User.3" user)
+		(45 "User.4" user)
+	)
+	(setup
+		(stackup
+			(layer "F.SilkS"
+				(type "Top Silk Screen")
+			)
+			(layer "F.Paste"
+				(type "Top Solder Paste")
+			)
+			(layer "F.Mask"
+				(type "Top Solder Mask")
+				(thickness 0.01)
+			)
+			(layer "F.Cu"
+				(type "copper")
+				(thickness 0.035)
+			)
+			(layer "dielectric 1"
+				(type "core")
+				(thickness 1.51)
+				(material "FR4")
+				(epsilon_r 4.5)
+				(loss_tangent 0.02)
+			)
+			(layer "B.Cu"
+				(type "copper")
+				(thickness 0.035)
+			)
+			(layer "B.Mask"
+				(type "Bottom Solder Mask")
+				(thickness 0.01)
+			)
+			(layer "B.Paste"
+				(type "Bottom Solder Paste")
+			)
+			(layer "B.SilkS"
+				(type "Bottom Silk Screen")
+			)
+			(copper_finish "None")
+			(dielectric_constraints no)
+		)
+		(pad_to_mask_clearance 0)
+		(allow_soldermask_bridges_in_footprints no)
+		(tenting
+			(front yes)
+			(back yes)
+		)
+		(covering
+			(front no)
+			(back no)
+		)
+		(plugging
+			(front no)
+			(back no)
+		)
+		(capping no)
+		(filling no)
+		(zone_defaults)
+		(pcbplotparams
+			(layerselection 0x00000000_00000000_55555555_5755f5ff)
+			(plot_on_all_layers_selection 0x00000000_00000000_00000000_00000000)
+			(disableapertmacros no)
+			(usegerberextensions no)
+			(usegerberattributes yes)
+			(usegerberadvancedattributes yes)
+			(creategerberjobfile yes)
+			(dashed_line_dash_ratio 12)
+			(dashed_line_gap_ratio 3)
+			(svgprecision 4)
+			(plotframeref no)
+			(mode 1)
+			(useauxorigin no)
+			(pdf_front_fp_property_popups yes)
+			(pdf_back_fp_property_popups yes)
+			(pdf_metadata yes)
+			(pdf_single_document no)
+			(dxfpolygonmode yes)
+			(dxfimperialunits yes)
+			(dxfusepcbnewfont yes)
+			(psnegative no)
+			(psa4output no)
+			(plot_black_and_white yes)
+			(sketchpadsonfab no)
+			(plotpadnumbers no)
+			(hidednponfab no)
+			(sketchdnponfab yes)
+			(crossoutdnponfab yes)
+			(subtractmaskfromsilk no)
+			(outputformat 1)
+			(mirror no)
+			(drillshape 1)
+			(scaleselection 1)
+			(outputdirectory "")
+		)
+	)
+	(embedded_fonts no)
+)

Commit message: Lay out one row
Parts:
- added BZ1: Buzzer, Buzzer_Beeper:MagneticBuzzer_StarMicronics_QMB-105, F.Cu at (51.1, 94.3)
- added C100: 100n, Capacitor_SMD:C_0402_1005Metric, F.Cu at (34.0, 71.0)
- added C101: 100n, Capacitor_SMD:C_0402_1005Metric, F.Cu at (46.5, 71.0)
- added C102: 100n, Capacitor_SMD:C_0402_1005Metric, F.Cu at (59.0, 71.0)
- added C103: 100n, Capacitor_SMD:C_0402_1005Metric, F.Cu at (71.5, 71.0)
- added C104: 100n, Capacitor_SMD:C_0402_1005Metric, F.Cu at (84.0, 71.0)
- added D100: WS2812B, Local:LED_ARGB_5050, F.Cu at (30.0, 70.0)
- added D101: WS2812B, Local:LED_ARGB_5050, F.Cu at (42.5, 70.0)
- added D102: WS2812B, Local:LED_ARGB_5050, F.Cu at (55.0, 70.0)
- added D103: WS2812B, Local:LED_ARGB_5050, F.Cu at (67.5, 70.0)
- added D104: WS2812B, Local:LED_ARGB_5050, F.Cu at (80.0, 70.0)
- added J1: Arduino Nano SuperMini, Local:DevBoard_SuperMini, F.Cu at (35.7, 94.4)
- added SW0: SW_Push, Button_Switch_SMD:SW_Push_1TS009xxxx-xxxx-xxxx_6x6x5mm, F.Cu at (76.2, 85.9)
- added SW1: SW_Push, Button_Switch_SMD:SW_Push_1TS009xxxx-xxxx-xxxx_6x6x5mm, F.Cu at (84.6, 93.9)
- added SW2: SW_Push, Button_Switch_SMD:SW_Push_1TS009xxxx-xxxx-xxxx_6x6x5mm, F.Cu at (76.3, 102.6)
- added SW3: SW_Push, Button_Switch_SMD:SW_Push_1TS009xxxx-xxxx-xxxx_6x6x5mm, F.Cu at (67.2, 94.2)
Routing:
- net Net-(D100-DOUT): track 0.00 -> 17.9 mm
- net +5V: track 0.00 -> 11.6 mm, vias 0 -> 6
- net Net-(D102-DOUT): track 0.00 -> 8.97 mm
- net Net-(D101-DOUT): track 0.00 -> 8.97 mm
- net Net-(D103-DOUT): track 0.00 -> 8.97 mm
- net GND: vias 0 -> 11
- added copper zone on B.Cu, net GND
- added copper zone on F.Cu, net GND
