File: Snail/Snail.kicad_sch (KiCad schematic)
At the start: 0 parts

Commit message: 🚧 Schematic, lights TO-DO
Parts:
- added BZ1: Buzzer, Buzzer_Beeper:MagneticBuzzer_StarMicronics_QMB-105, symbol Device:Buzzer
- added D1: 1N5819, Diode_SMD:D_SOD-323, symbol Device:D
- added J1: Arduino Nano SuperMini, Local:DevBoard_SuperMini, symbol Connector_Generic:Conn_02x09_Counter_Clockwise
- added Q1: MMBT3904, Package_TO_SOT_SMD:SOT-23, symbol Transistor_BJT:MMBT3904
- added R1: 4.7k, Resistor_SMD:R_0402_1005Metric, symbol Device:R
- added R2: 10, Resistor_SMD:R_0402_1005Metric, symbol Device:R
- added SW1, SW2, SW3, SW4: SW_Push, Button_Switch_SMD:SW_Push_1TS009xxxx-xxxx-xxxx_6x6x5mm, symbol Switch:SW_Push
Connections:
- new net: BZ1.1 (+), D1.1 (K), R2.2
- new net: BZ1.2 (-), D1.2 (A), Q1.3 (C)
- new net: Q1.1 (B), R1.2
- new net +5V: J1.16 (Pin_16), R2.1
- new net BUZZER: J1.6 (Pin_6), R1.1
- new net GND: J1.17 (Pin_17), Q1.2 (E), SW1.2, SW2.2, SW3.2, SW4.2
- new net KEY_1: J1.12 (Pin_12), SW1.1
- new net KEY_2: J1.13 (Pin_13), SW2.1
- new net KEY_3: J1.14 (Pin_14), SW3.1
- new net KEY_4: J1.15 (Pin_15), SW4.1
- new net LIGHT_SD: J1.4 (Pin_4)
- no-connect marks 0 -> 10
Other:
- added sheet LEDs (LEDs.kicad_sch)
- note added: "A0"
- note added: "A1"
- note added: "A2"
- note added: "A3"
- note added: "A4"
- note added: "A5"
- note added: "D0"
- note added: "D1"
- note added: "D2"
- note added: "D3"
- note added: "D4"
- note added: "D5"
- note added: "D6"
- note added: "D7"
- note added: "D8"
- note added: "LDO 5V"
- note added: "RX"
- note added: "TX"
- note added: "VIN"

Commit message: Full schematic & footprints
Parts:
- added C1, C2: 10u, Capacitor_SMD:C_0603_1608Metric, symbol Device:C
- added C100, C101, C102, C103, C104, C105, C106, C107, C108, C109, C110, C111, C112, C113, C114, C115, C116, C117, C118, C119, C120, C121, C122, C123, C124, C125, C126, C127, C128, C129, C130, C131, C132, C133, C134, C135, C136, C137: 100n, Capacitor_SMD:C_0402_1005Metric, symbol Device:C
- added D100, D101, D102, D103, D104, D105, D106, D107, D108, D109, D110, D111, D112, D113, D114, D115, D116, D117, D118, D119, D120, D121, D122, D123, D124, D125, D126, D127, D128, D129, D130, D131, D132, D133, D134: WS2812B, Local:LED_ARGB_5050, symbol LED:WS2812B
- added D135, D136, D137: WS2812B, Local:LED_ARGB_3528, symbol LED:WS2812B
- renumbered SW1 to SW0, SW2 to SW1, SW3 to SW2, SW4 to SW3
Connections:
- net KEY_4 is gone; now on net KEY_3: J1.15 (Pin_15), SW3.1
- net +5V: now also C1.1, C100.1, C101.1, C102.1, C103.1, C104.1, C105.1, C106.1, C107.1, C108.1, C109.1, C110.1, C111.1, C112.1, C113.1, C114.1, C115.1, C116.1, C117.1, C118.1, C119.1, C120.1, C121.1, C122.1, C123.1, C124.1, C125.1, C126.1, C127.1, C128.1, C129.1, C130.1, C131.1, C132.1, C133.1, C134.1, C135.1, C136.1, C137.1, C2.1, D100.1 (VDD), D101.1 (VDD), D102.1 (VDD), D103.1 (VDD), D104.1 (VDD), D105.1 (VDD), D106.1 (VDD), D107.1 (VDD), D108.1 (VDD), D109.1 (VDD), D110.1 (VDD), D111.1 (VDD), D112.1 (VDD), D113.1 (VDD), D114.1 (VDD), D115.1 (VDD), D116.1 (VDD), D117.1 (VDD), D118.1 (VDD), D119.1 (VDD), D120.1 (VDD), D121.1 (VDD), D122.1 (VDD), D123.1 (VDD), D124.1 (VDD), D125.1 (VDD), D126.1 (VDD), D127.1 (VDD), D128.1 (VDD), D129.1 (VDD), D130.1 (VDD), D131.1 (VDD), D132.1 (VDD), D133.1 (VDD), D134.1 (VDD), D135.1 (VDD), D136.1 (VDD), D137.1 (VDD)
- net GND: now also C1.2, C100.2, C101.2, C102.2, C103.2, C104.2, C105.2, C106.2, C107.2, C108.2, C109.2, C110.2, C111.2, C112.2, C113.2, C114.2, C115.2, C116.2, C117.2, C118.2, C119.2, C120.2, C121.2, C122.2, C123.2, C124.2, C125.2, C126.2, C127.2, C128.2, C129.2, C130.2, C131.2, C132.2, C133.2, C134.2, C135.2, C136.2, C137.2, C2.2, D100.3 (VSS), D101.3 (VSS), D102.3 (VSS), D103.3 (VSS), D104.3 (VSS), D105.3 (VSS), D106.3 (VSS), D107.3 (VSS), D108.3 (VSS), D109.3 (VSS), D110.3 (VSS), D111.3 (VSS), D112.3 (VSS), D113.3 (VSS), D114.3 (VSS), D115.3 (VSS), D116.3 (VSS), D117.3 (VSS), D118.3 (VSS), D119.3 (VSS), D120.3 (VSS), D121.3 (VSS), D122.3 (VSS), D123.3 (VSS), D124.3 (VSS), D125.3 (VSS), D126.3 (VSS), D127.3 (VSS), D128.3 (VSS), D129.3 (VSS), D130.3 (VSS), D131.3 (VSS), D132.3 (VSS), D133.3 (VSS), D134.3 (VSS), D135.3 (VSS), D136.3 (VSS), D137.3 (VSS)
- net KEY_1: now also J1.13 (Pin_13), SW1.1; no longer J1.12 (Pin_12), SW0.1
- net KEY_2: now also J1.14 (Pin_14), SW2.1; no longer J1.13 (Pin_13), SW1.1
- net KEY_3: no longer J1.14 (Pin_14), SW2.1
- net LIGHT_SD: now also D100.4 (DIN)
- new net: D115.2 (DOUT), D116.4 (DIN)
- new net: D114.2 (DOUT), D115.4 (DIN)
- new net: D129.2 (DOUT), D130.4 (DIN)
- new net: D128.2 (DOUT), D129.4 (DIN)
- new net: D130.2 (DOUT), D131.4 (DIN)
- new net: D107.2 (DOUT), D108.4 (DIN)
- new net: D106.2 (DOUT), D107.4 (DIN)
- new net: D132.2 (DOUT), D133.4 (DIN)
- new net: D131.2 (DOUT), D132.4 (DIN)
- new net: D102.2 (DOUT), D103.4 (DIN)
- new net: D101.2 (DOUT), D102.4 (DIN)
- new net: D120.2 (DOUT), D121.4 (DIN)
- new net: D119.2 (DOUT), D120.4 (DIN)
- new net: D111.2 (DOUT), D112.4 (DIN)
- new net: D110.2 (DOUT), D111.4 (DIN)
- new net: D127.2 (DOUT), D128.4 (DIN)
- new net: D126.2 (DOUT), D127.4 (DIN)
- new net: D100.2 (DOUT), D101.4 (DIN)
- new net: D104.2 (DOUT), D105.4 (DIN)
- new net: D103.2 (DOUT), D104.4 (DIN)
- new net: D113.2 (DOUT), D114.4 (DIN)
- new net: D133.2 (DOUT), D134.4 (DIN)
- new net: D125.2 (DOUT), D126.4 (DIN)
- new net: D124.2 (DOUT), D125.4 (DIN)
- new net: D109.2 (DOUT), D110.4 (DIN)
- new net: D108.2 (DOUT), D109.4 (DIN)
- new net: D136.2 (DOUT), D137.4 (DIN)
- new net: D135.2 (DOUT), D136.4 (DIN)
- new net: D105.2 (DOUT), D106.4 (DIN)
- new net: D123.2 (DOUT), D124.4 (DIN)
- new net: D122.2 (DOUT), D123.4 (DIN)
- new net: D116.2 (DOUT), D117.4 (DIN)
- new net: D112.2 (DOUT), D113.4 (DIN)
- new net: D118.2 (DOUT), D119.4 (DIN)
- new net: D117.2 (DOUT), D118.4 (DIN)
- new net: D134.2 (DOUT), D135.4 (DIN)
- new net: D121.2 (DOUT), D122.4 (DIN)
- new net KEY_0: J1.12 (Pin_12), SW0.1
- no-connect marks 10 -> 11
Other:
- removed sheet LEDs
- moved on the sheet: BZ1, D1, Q1, R1, R2

Commit message: Finish layout & routing
Connections:
- net BUZZER: now also J1.15 (Pin_15); no longer J1.6 (Pin_6)
- net KEY_0: now also J1.10 (Pin_10); no longer J1.12 (Pin_12)
- net KEY_1: now also J1.8 (Pin_8); no longer J1.13 (Pin_13)
- net KEY_2: now also J1.9 (Pin_9); no longer J1.14 (Pin_14)
- net KEY_3: now also J1.11 (Pin_11); no longer J1.15 (Pin_15)

Commit message: hw: Update files with actual mounted component value
Parts:
- R2: value 10 -> 220
Other:
- note added: "16 Ω, 30 mA"
Changed lines of the file:
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@@
 		)
 	)
+	(text "16 Ω, 30 mA"
+		(exclude_from_sim no)
+		(at 87.63 88.9 0)
+		(effects
+			(font
+				(size 1.27 1.27)
+				(italic yes)
+			)
+			(justify right)
+		)
+	)
 	(text "A2"
 		(exclude_from_sim no)
@@
 			)
 		)
-		(property "Value" "10"
+		(property "Value" "220"
 			(at 91.44 77.4699 0)
 			(show_name no)
