File: Snail/libs/Local.kicad_blocks/LED_Row.kicad_block/LED_Row.kicad_pcb (KiCad board)
At the start: 2 copper layers, 10 parts

Commit message: Finish layout & routing
Parts:
- moved C100 134.9 mm to (74.0, 199.8)
- moved C101 134.9 mm to (86.5, 199.8)
- moved C102 134.9 mm to (99.0, 199.8)
- moved C103 134.9 mm to (111.5, 199.8)
- moved C104 134.9 mm to (124.0, 199.8)
- moved D100 134.9 mm to (70.0, 198.8)
- moved D101 134.9 mm to (82.5, 198.8)
- moved D102 134.9 mm to (95.0, 198.8)
- moved D103 134.9 mm to (107.5, 198.8)
- moved D104 134.9 mm to (120.0, 198.8)
Routing:
- net Net-(D100-DOUT): track 17.9 -> 8.97 mm
- net GND: vias 11 -> 10
